File: pcb/SensEdu.kicad_sch (KiCad schematic)
At the start: 26 parts, among them J1 Power, J10 Barrel_Jack_Switch, J13 Conn_02x01, J14 Conn_02x01, J15 Conn_02x01, J18 Conn_03x01, J2 PWM, J3 Analog, J4 PWM, J5 Analog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

Commit message: feat: Fix DRC errors and warnings
Updated footprint links
Updated schematic symbol for LT1790 to remove warnings
Parts:
- J7: footprint (none) -> Connector_PinSocket_2.54mm:PinSocket_2x18_P2.54mm_Vertical
Changed lines of the file:
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@@
 			)
 		)
-		(property "Footprint" ""
+		(property "Footprint" "Connector_PinSocket_2.54mm:PinSocket_2x18_P2.54mm_Vertical"
 			(at 115.57 130.81 0)
 			(effects
