File: pcb/_autosave-SensEdu.kicad_pcb (KiCad board)
At the start: 4 copper layers, 99.1 x 54 mm, 147 parts, among them J1 Power, J10 Barrel_Jack_Switch, J11 Conn_01x04_Pin, J12 Conn_01x04_Pin, J13 Conn_02x01, J14 Conn_02x01, J15 Conn_02x01, J16 Conn_02x01, J17 Conn_03x01, J18 Conn_03x01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

Commit message: feat: Fix DRC errors and warnings
Updated footprint links
Updated schematic symbol for LT1790 to remove warnings
Parts:
- LS1, LS2: value Speaker_Ultrasound -> 328ST16M; footprint Speaker:328ST16M_Speaker -> SensEdu:328ST16M_Speaker
- U4, U7: value R_8_ADI -> ADA4891
