File: pcb/General_pupose_Amplifiers.kicad_sch (KiCad schematic)
At the start: 36 parts, among them J10 Conn_01x04_Pin, J11 Conn_01x04_Pin, J8 Conn_01x04_Pin, J9 Conn_01x04_Pin, U6 AD8426ACPZ-R7, U7 AD8426ACPZ-R7

Commit message: pcb routing finished
very messy
Connections:
- net out+: no longer J10.2 (Pin_2), J8.2 (Pin_2), J9.2 (Pin_2), R20.1, R24.1, R27.1
- net out-: no longer J10.3 (Pin_3), J8.3 (Pin_3), J9.3 (Pin_3), R19.1, R22.1, R26.1
- new net: J8.2 (Pin_2), R20.1
- new net: J8.3 (Pin_3), R19.1
- new net: J9.2 (Pin_2), R24.1
- new net: J9.3 (Pin_3), R22.1
- new net: J10.2 (Pin_2), R27.1
- new net: J10.3 (Pin_3), R26.1
Changed lines of the file:
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@@
-		)
-	)
-	(label "out+"
-		(at 38.1 39.37 0)
-		(effects
-			(font
-				(size 1.27 1.27)
-			)
-			(justify left bottom)
-		)
-	)
-	(label "out+"
-		(at 107.442 39.37 0)
-		(effects
-			(font
-				(size 1.27 1.27)
-			)
-			(justify left bottom)
 		)
 	)
@@
 		(effects
 			(font
-				(size 1.27 1.27)
-			)
-			(justify left bottom)
-		)
-	)
-	(label "out-"
-		(at 38.1 41.91 0)
-		(effects
-			(font
-				(size 1.27 1.27)
-			)
-			(justify left bottom)
-		)
-	)
-	(label "out+"
-		(at 172.72 39.37 0)
-		(effects
-			(font
-				(size 1.27 1.27)
-			)
-			(justify left bottom)
-		)
-	)
-	(label "out-"
-		(at 107.442 41.91 0)
-		(effects
-			(font
-				(size 1.27 1.27)
-			)
-			(justify left bottom)
-		)
-	)
-	(label "out-"
-		(at 172.72 41.91 0)
-		(effects
-			(font

Commit message: in works
Other:
- title: SensEdu 0.7 -> SensEdu 0.9
Changed lines of the file:
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@@
 	(paper "A4")
 	(title_block
-		(title "SensEdu 0.7")
+		(title "SensEdu 0.9")
 		(date "2025-12-05")
 		(company "Infineon Technologies")
