File: pcb/External_Microphone_Connectors.kicad_sch (KiCad schematic)
At the start: 36 parts, among them J10 Conn_01x04_Pin, J11 Conn_01x04_Pin, J8 Conn_01x04_Pin, J9 Conn_01x04_Pin, U6 AD8426ACPZ-R7, U7 AD8426ACPZ-R7

Commit message: feat: Redraw PCB layout
- Change supply polarity and pin numbers of ADA4511
- Change cap of switches to 100n to reduce bom
- Change supply of sensors to unison 3.3V
- Rearrange mic and amps pins
- Add mountains
- Add Infineon logo
Parts:
- added C61, C62: 1u, Capacitor_SMD:C_0603_1608Metric, symbol SensEdu:C
- C30: renamed from C34; footprint Capacitor_SMD:C_0805_2012Metric -> Capacitor_SMD:C_0603_1608Metric; symbol Device:C -> SensEdu:C
- C31: renamed from C39; footprint Capacitor_SMD:C_0805_2012Metric -> Capacitor_SMD:C_0603_1608Metric; symbol Device:C -> SensEdu:C
- C32: renamed from C43; footprint Capacitor_SMD:C_0805_2012Metric -> Capacitor_SMD:C_0603_1608Metric; symbol Device:C -> SensEdu:C
- C33: renamed from C47; footprint Capacitor_SMD:C_0805_2012Metric -> Capacitor_SMD:C_0603_1608Metric; symbol Device:C -> SensEdu:C
- C34: renamed from C37; footprint Capacitor_SMD:C_0805_2012Metric -> Capacitor_SMD:C_0603_1608Metric; symbol Device:C -> SensEdu:C
- C35: renamed from C45; footprint Capacitor_SMD:C_0805_2012Metric -> Capacitor_SMD:C_0603_1608Metric; symbol Device:C -> SensEdu:C
- C36: renamed from C41; footprint Capacitor_SMD:C_0805_2012Metric -> Capacitor_SMD:C_0603_1608Metric; symbol Device:C -> SensEdu:C
- C37: renamed from C32; footprint Capacitor_SMD:C_0805_2012Metric -> Capacitor_SMD:C_0603_1608Metric; symbol Device:C -> SensEdu:C
- C38: renamed from C35; footprint Capacitor_SMD:C_0805_2012Metric -> Capacitor_SMD:C_0603_1608Metric; symbol Device:C -> SensEdu:C
- C39: renamed from C38; footprint Capacitor_SMD:C_0805_2012Metric -> Capacitor_SMD:C_0603_1608Metric; symbol Device:C -> SensEdu:C
- C40: renamed from C44; footprint Capacitor_SMD:C_0805_2012Metric -> Capacitor_SMD:C_0603_1608Metric; symbol Device:C -> SensEdu:C
- C41: renamed from C46; footprint Capacitor_SMD:C_0805_2012Metric -> Capacitor_SMD:C_0603_1608Metric; symbol Device:C -> SensEdu:C
- C42: renamed from C40; footprint Capacitor_SMD:C_0805_2012Metric -> Capacitor_SMD:C_0603_1608Metric; symbol Device:C -> SensEdu:C
- C43: renamed from C42; footprint Capacitor_SMD:C_0805_2012Metric -> Capacitor_SMD:C_0603_1608Metric; symbol Device:C -> SensEdu:C
- C44: renamed from C30; footprint Capacitor_SMD:C_0805_2012Metric -> Capacitor_SMD:C_0603_1608Metric; symbol Device:C -> SensEdu:C
- C45: renamed from C33; footprint Capacitor_SMD:C_0805_2012Metric -> Capacitor_SMD:C_0603_1608Metric; symbol Device:C -> SensEdu:C
- C46: renamed from C31; footprint Capacitor_SMD:C_0805_2012Metric -> Capacitor_SMD:C_0603_1608Metric; symbol Device:C -> SensEdu:C
- C47: renamed from C36; footprint Capacitor_SMD:C_0805_2012Metric -> Capacitor_SMD:C_0603_1608Metric; symbol Device:C -> SensEdu:C
- J10, J11, J8, J9: symbol Connector:Conn_01x04_Pin -> SensEdu:Conn_01x04_Pin
- R18: renamed from R19; footprint Resistor_SMD:R_0805_2012Metric -> Resistor_SMD:R_0603_1608Metric; symbol Device:R -> SensEdu:R
- R19: renamed from R20; footprint Resistor_SMD:R_0805_2012Metric -> Resistor_SMD:R_0603_1608Metric; symbol Device:R -> SensEdu:R
- R20: renamed from R22; footprint Resistor_SMD:R_0805_2012Metric -> Resistor_SMD:R_0603_1608Metric; symbol Device:R -> SensEdu:R
- R21: renamed from R24; footprint Resistor_SMD:R_0805_2012Metric -> Resistor_SMD:R_0603_1608Metric; symbol Device:R -> SensEdu:R
- R22: renamed from R26; footprint Resistor_SMD:R_0805_2012Metric -> Resistor_SMD:R_0603_1608Metric; symbol Device:R -> SensEdu:R
- R23: renamed from R27; footprint Resistor_SMD:R_0805_2012Metric -> Resistor_SMD:R_0603_1608Metric; symbol Device:R -> SensEdu:R
- R24: renamed from R28; footprint Resistor_SMD:R_0805_2012Metric -> Resistor_SMD:R_0603_1608Metric; symbol Device:R -> SensEdu:R
- R25: renamed from R29; footprint Resistor_SMD:R_0805_2012Metric -> Resistor_SMD:R_0603_1608Metric; symbol Device:R -> SensEdu:R
- R26: renamed from R18; footprint Resistor_SMD:R_0805_2012Metric -> Resistor_SMD:R_0603_1608Metric; symbol Device:R -> SensEdu:R
- R27: renamed from R21; footprint Resistor_SMD:R_0805_2012Metric -> Resistor_SMD:R_0603_1608Metric; symbol Device:R -> SensEdu:R
- R28: renamed from R23; footprint Resistor_SMD:R_0805_2012Metric -> Resistor_SMD:R_0603_1608Metric; symbol Device:R -> SensEdu:R
- R29: renamed from R25; footprint Resistor_SMD:R_0805_2012Metric -> Resistor_SMD:R_0603_1608Metric; symbol Device:R -> SensEdu:R
- U6: symbol SensEdu:AD8426ACPZ-R7 -> SensEdu:AD8426ACPZ-R7_1
Connections:
- net mic7_out1 is gone; now on net amp3_out_P: C36.1, C43.2, R23.2
- net mic7_out2 is gone; now on net amp3_out_N: C36.2, C42.2, R22.2
- net +3.3V: now also C61.1, C62.1
- net GND: now also C61.2, C62.2
- net MIC5_OUT renamed AMP1_EXT_OUT
- net MIC6_OUT renamed AMP2_EXT_OUT
- net MIC7_OUT renamed AMP3_EXT_OUT
- net MIC8_OUT renamed AMP4_EXT_OUT
- net mic2_out1 renamed amp3_out_P
- net mic2_out2 renamed amp3_out_N
- net mic3_out1 renamed amp1_out_P
- net amp1_out_P: now also C37.1, C45.2, R19.2
- net mic3_out2 renamed amp1_out_N
- net amp1_out_N: now also C37.2, C44.2, R18.2
- removed net mic5_out1: C37.1, C45.2, R19.2, U6.9 (+IN2)
- removed net mic5_out2: C37.2, C44.2, R18.2, U6.12 (-IN2)
- net mic6_out1 renamed amp2_out_P
- net amp2_out_P: now also U6.9 (+IN2)
- net mic6_out2 renamed amp2_out_N
- net amp2_out_N: now also U6.12 (-IN2)
- net mic8_out1 renamed amp4_out_P
- net mic8_out2 renamed amp4_out_N
Other:
- moved on the sheet: C34, C35, C36, C38, C39, C40, C41, C42, C43, R26, R29

Commit message: refactor: Update PDF and information
- Add BOM
Other:
- title: SensEdu 0.9 -> SensEdu
Changed lines of the file:
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@@
 	(paper "A4")
 	(title_block
-		(title "SensEdu 0.9")
-		(date "2025-12-05")
+		(title "SensEdu")
+		(date "2026-02-26")
 		(rev "0.9")
 		(company "Infineon Technologies")

Commit message: feat: Improve PCB design after tests of rev 0.8
- Added new generation of humidity sensor
- New silkscreen information for different components
- Added additional testpoints
- Removed PWM path for ultrasound transmitter
Parts:
- C30, C31, C32, C33, C36, C42, C43: footprint Capacitor_SMD:C_0603_1608Metric -> SensEdu:C_0603_1608Metric
- C34: renamed from C37; footprint Capacitor_SMD:C_0603_1608Metric -> SensEdu:C_0603_1608Metric
- C35: renamed from C34; footprint Capacitor_SMD:C_0603_1608Metric -> SensEdu:C_0603_1608Metric
- C37: renamed from C35; footprint Capacitor_SMD:C_0603_1608Metric -> SensEdu:C_0603_1608Metric
- C38: renamed from C44; footprint Capacitor_SMD:C_0603_1608Metric -> SensEdu:C_0603_1608Metric
- C39: renamed from C45; footprint Capacitor_SMD:C_0603_1608Metric -> SensEdu:C_0603_1608Metric
- C40: renamed from C38; footprint Capacitor_SMD:C_0603_1608Metric -> SensEdu:C_0603_1608Metric
- C41: renamed from C39; footprint Capacitor_SMD:C_0603_1608Metric -> SensEdu:C_0603_1608Metric
- C44: renamed from C40; footprint Capacitor_SMD:C_0603_1608Metric -> SensEdu:C_0603_1608Metric
- C45: renamed from C41; footprint Capacitor_SMD:C_0603_1608Metric -> SensEdu:C_0603_1608Metric
- C46: renamed from C61; footprint Capacitor_SMD:C_0603_1608Metric -> SensEdu:C_0603_1608Metric
- C47: renamed from C46; footprint Capacitor_SMD:C_0603_1608Metric -> SensEdu:C_0603_1608Metric
- C48: renamed from C62; footprint Capacitor_SMD:C_0603_1608Metric -> SensEdu:C_0603_1608Metric
- C49: renamed from C47; footprint Capacitor_SMD:C_0603_1608Metric -> SensEdu:C_0603_1608Metric
- J10, J11, J8, J9: footprint Connector_PinSocket_2.54mm:PinSocket_1x04_P2.54mm_Vertical -> SensEdu:PinSocket_1x04_P2.54mm_Vertical
- R18, R19, R20, R21, R22, R23, R24, R25, R26, R27, R28, R29: footprint Resistor_SMD:R_0603_1608Metric -> SensEdu:R_0603_1608Metric
