File: projects/Ultrasonic_3D_Tracking/pcbs/sensedu-extended-kicad/General_pupose_Amplifiers.kicad_sch (KiCad schematic)
At the start: 36 parts, among them J11 Conn_01x04_Pin, U1 AD8426ACPZ-R7, U2 AD8426ACPZ-R7

Commit message: Fix: Cleaned schematic
- project is not correctly set up, so cannot be ordered without further
   work
Parts:
- renumbered C1 to C62, C1 to C63, C1 to C64, C1 to C65, C1 to C66, C1 to C67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
