File: projects/Ultrasonic_3D_Tracking/pcbs/sensedu-extended-kicad/Speakers.kicad_sch (KiCad schematic)
At the start: 34 parts, among them J17 Conn_03x01, U4 ADA4891, U7 ADA4891

Commit message: Fix: Cleaned schematic
- project is not correctly set up, so cannot be ordered without further
   work
Parts:
- renumbered C1 to C47, C1 to C48, C1 to C49, C1 to C50, C1 to C51, C1 to C52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
