File: projects/Ultrasonic_3D_Tracking/pcbs/sensedu-extended-kicad/Ultrasound shield_8mic.kicad_pcb (KiCad board)
At the start: 4 copper layers, 199 x 200 mm, 183 parts, among them J1 Power, J10 Barrel_Jack_Switch, J11 Conn_01x04_Pin, J12 Conn_01x04_Pin, J13 Conn_02x01, J14 Conn_02x01, J15 Conn_02x01, J16 Conn_02x01, J17 Conn_03x01, J18 Conn_03x01, J19 Conn_03x01, J2 PWM, J20 Conn_01x04_Pin, J3 Analog, J4 PWM, J5 Analog, J6 Communication, J7 Digital, J8 Conn_03x01, J9 Conn_01x04_Pin, U1 AD8426ACPZ-R7, U10 AD8426ACPZ-R7, U12 TLS850C2TE_V33, U13 NCP1117-2.5_SOT223, U2 AD8426ACPZ-R7, U3 LT1790ACS6-1.25, U4 R_8_ADI, U5 AD8426ACPZ-R7, U6 AD8426ACPZ-R7, U7 R_8_ADI, U8 DPS310XTSA1, U9 AD8426ACPZ-R7

Commit message: pcb: Update references
Parts:
- U8: renamed from U7; value R_8_ADI -> ADA4891
- U9: renamed from U4; value R_8_ADI -> ADA4891
- renumbered C38 to C1, C30 to C10, C13 to C11, C8 to C12, C31 to C13, C7 to C14, C14 to C15, C11 to C16, C28 to C17, C12 to C18, C29 to C19, C3 to C2, C1 to C20, C5 to C21, C6 to C22, C9 to C23, C20 to C24, C2 to C25, C16 to C26, C17 to C27, C18 to C28, C19 to C29, C4 to C3, C66 to C30, C67 to C31, C68 to C32, C78 to C33, C59 to C34, C69 to C35, C70 to C36, C71 to C37, C60 to C38, C72 to C39, C36 to C4, C73 to C40, C74 to C41, C79 to C42, C65 to C43, C75 to C44, C76 to C45, C77 to C46, C27 to C47, C25 to C48, C21 to C49, C37 to C5, C23 to C50, C24 to C51, C26 to C52, C22 to C53, C39 to C54, C63 to C55, C43 to C56, C32 to C57, C34 to C58, C35 to C59, C55 to C6, C64 to C60, C15 to C61, C33 to C62, C44 to C63, C45 to C64, C46 to C65, C61 to C66, C40 to C67, C47 to C68, C48 to C69, C56 to C7, C49 to C70, C41 to C71, C50 to C72, C51 to C73, C52 to C74, C62 to C75, C42 to C76, C53 to C77, C54 to C78, C58 to C79, C57 to C8, C10 to C9, J18 to J1, J5 to J10, J6 to J11, J7 to J12, J16 to J13, J17 to J14, J8 to J15, J19 to J16, J9 to J17, J11 to J18, J12 to J19, J15 to J2, J13 to J3, J10 to J4, J2 to J5, J1 to J6, J14 to J7, J3 to J8, J4 to J9, R9 to R10, R10 to R11, R13 to R12, R11 to R13, R43 to R14, R51 to R15, R44 to R16, R45 to R17, R52 to R18, R46 to R19, R4 to R2, R47 to R20, R53 to R21, R48 to R22, R49 to R23, R54 to R24, R50 to R25, R16 to R26, R17 to R27, R18 to R28, R20 to R29, R2 to R3, R19 to R30, R15 to R31, R14 to R32, R21 to R33, R22 to R34, R25 to R35, R5 to R4, R23 to R43, R32 to R44, R24 to R45, R26 to R46, R33 to R47, R27 to R48, R28 to R49, R3 to R5, R34 to R50, R29 to R51, R30 to R52, R35 to R53, R31 to R54, R7 to R6, R6 to R7, R12 to R9, U12 to U1, U8 to U10, U5 to U11, U6 to U12, U13 to U2, U1 to U4, U2 to U5, U9 to U6, U10 to U7
Connections:
- net Net-(J1-Pin_5) renamed /5V
- J10 pad 7: unconnected-(J5-Pin_7-Pad7) -> /A14
- J10 pad 8: unconnected-(J5-Pin_8-Pad8) -> /A15
- J6 pad 4: unconnected-(J1-Pin_4-Pad4) -> /3V3
